Commit message: 增加相机urdf

File: src/robot_description/urdf/seed_robot.urdf.xacro (robot description, xacro)
@@ -5,4 +5,5 @@
   <xacro:property name="white_color" value="1 1 1 1" />
   <xacro:property name="package_name" value="robot_description" />
+  <xacro:property name="camera_mesh_path" value="package://robot_description/meshes/gemini335_336/" />
   <!-- Material definitions -->
   <material name="base_material">
@@ -11,4 +12,13 @@
   <material name="white_material">
     <color rgba="${white_color}" />
+  </material>
+  <material name="camera_material">
+    <color rgba="1 1 1 1" />
+  </material>
+  <material name="camera_screw_material">
+    <color rgba="0.792156862745098 0.819607843137255 0.933333333333333 1" />
+  </material>
+  <material name="camera_sensor_material">
+    <color rgba="0.501960784313725 0.250980392156863 0.250980392156863 1" />
   </material>
   <!-- Macro for link with mesh -->
@@ -55,4 +65,5 @@
     </joint>
   </xacro:macro>
+  <!-- ====================== ROBOT ARM DEFINITION ====================== -->
   <!-- Base link -->
   <xacro:link_with_mesh
@@ -82,5 +93,5 @@
     izz="0.19723"
     origin_xyz="0 0 0"
-    origin_rpy="0 0 1" />
+    origin_rpy="0 0 0" />
   <!-- Joint 1 -->
   <xacro:revolute_joint
@@ -225,59 +236,284 @@
     effort="0"
     velocity="0" />
-  <!-- ros2_control configuration -->
-  <ros2_control name="FakeSystem" type="system">
-    <hardware>
-      <plugin>fake_components/GenericSystem</plugin>
-      <param name="fake_sensor_commands">false</param>
-      <param name="state_following_offset">0.0</param>
-    </hardware>
-    <joint name="joint1">
-      <command_interface name="position">
-        <param name="min">-2.627</param>
-        <param name="max">2.617</param>
-      </command_interface>
-      <state_interface name="position"/>
-      <state_interface name="velocity"/>
-    </joint>
-    <joint name="joint2">
-      <command_interface name="position">
-        <param name="min">-1.134</param>
-        <param name="max">1.919</param>
-      </command_interface>
-      <state_interface name="position"/>
-      <state_interface name="velocity"/>
-    </joint>
-    <joint name="joint3">
-      <command_interface name="position">
-        <param name="min">-3.281</param>
-        <param name="max">0.471</param>
-      </command_interface>
-      <state_interface name="position"/>
-      <state_interface name="velocity"/>
-    </joint>
-    <joint name="joint4">
-      <command_interface name="position">
-        <param name="min">-2.914</param>
-        <param name="max">2.914</param>
-      </command_interface>
-      <state_interface name="position"/>
-      <state_interface name="velocity"/>
-    </joint>
-    <joint name="joint5">
-      <command_interface name="position">
-        <param name="min">-0.593</param>
-        <param name="max">3.63</param>
-      </command_interface>
-      <state_interface name="position"/>
-      <state_interface name="velocity"/>
-    </joint>
-    <joint name="joint6">
-      <command_interface name="position">
-        <param name="min">-4.712</param>
-        <param name="max">4.712</param>
-      </command_interface>
-      <state_interface name="position"/>
-      <state_interface name="velocity"/>
-    </joint>
-  </ros2_control>
+  <!-- ====================== CAMERA DEFINITION ====================== -->
+  <!-- Camera mount joint - connects camera to base_link -->
+  <joint name="camera_mount_joint" type="fixed">
+    <origin xyz="0.665 0.00 0.35" rpy="0 1.0 -2.47601" />
+    <parent link="base_link" />
+    <child link="camera_link" />
+  </joint>
+  <!-- Camera main link -->
+  <link name="camera_link">
+    <inertial>
+      <origin xyz="0.00277269933215555 -1.06084680351007E-05 0.012801025085723" rpy="0 0 0" />
+      <mass value="0.0186143499064346" />
+      <inertia ixx="1.38922229644605E-05" ixy="-4.74617876641156E-09"
+        ixz="1.99175628166615E-08"
+        iyy="1.70686808598814E-06" iyz="-7.18717290327325E-09" izz="1.31766831843134E-05" />
+    </inertial>
+    <visual>
+      <origin xyz="0 0 0" rpy="0 0 0" />
+      <geometry>
+        <mesh filename="${camera_mesh_path}camera_link.STL" />
+      </geometry>
+      <material name="camera_material" />
+    </visual>
+    <collision>
+      <origin xyz="0 0 0" rpy="0 0 0" />
+      <geometry>
+        <mesh filename="${camera_mesh_path}camera_link.STL" />
+      </geometry>
+    </collision>
+  </link>
+  <!-- Camera bottom screw frame -->
+  <link name="camera_bottom_screw_frame">
+    <inertial>
+      <origin xyz="0.00255168206289301 -0.00123934714960528 0.0118889875786098" rpy="0 0 0" />
+      <mass value="0.00564476880678651" />
+      <inertia ixx="3.07690693820862E-06" ixy="-1.85045956307764E-08"
+        ixz="-9.2792327175816E-09"
+        iyy="2.27632852811487E-07" iyz="1.65233162864392E-08" izz="2.93985735090777E-06" />
+    </inertial>
+    <visual>
+      <origin xyz="0 0 0" rpy="0 0 0" />
+      <geometry>
+        <mesh filename="${camera_mesh_path}camera_bottom_screw_frame.STL" />
+      </geometry>
+      <material name="camera_screw_material" />
+    </visual>
+    <collision>
+      <origin xyz="0 0 0" rpy="0 0 0" />
+      <geometry>
+        <mesh filename="${camera_mesh_path}camera_bottom_screw_frame.STL" />
+      </geometry>
+    </collision>
+  </link>
+  <joint name="camera_bottom_screw_frame_joint" type="fixed">
+    <origin xyz="0 0 0" rpy="0 0 0" />
+    <parent link="camera_link" />
+    <child link="camera_bottom_screw_frame" />
+  </joint>
+  <!-- Infrared camera 1 frame -->
+  <link name="camera_infra_1_frame">
+    <inertial>
+      <origin xyz="-0.00158020887627678 -1.52683853303637E-08 -1.4860800305164E-07" rpy="0 0 0" />
+      <mass value="0.000453168790516429" />
+      <inertia ixx="4.34108781911687E-09" ixy="-3.69655517007001E-13"
+        ixz="-1.45486421873185E-13"
+        iyy="4.84012226840139E-09" iyz="1.92888940614786E-14" izz="4.84044260907388E-09" />
+    </inertial>
+    <visual>
+      <origin xyz="0 0 0" rpy="0 0 0" />
+      <geometry>
+        <mesh filename="${camera_mesh_path}camera_infra_1_frame.STL" />
+      </geometry>
+      <material name="camera_sensor_material" />
+    </visual>
+    <collision>
+      <origin xyz="0 0 0" rpy="0 0 0" />
+      <geometry>
+        <mesh filename="${camera_mesh_path}camera_infra_1_frame.STL" />
+      </geometry>
+    </collision>
+  </link>
+  <joint name="camera_infra_1_joint" type="fixed">
+    <origin xyz="0.01587 -0.025 0.0125" rpy="0 0 0" />
+    <parent link="camera_bottom_screw_frame" />
+    <child link="camera_infra_1_frame" />
+  </joint>
+  <!-- Infrared camera 1 optical frame -->
+  <link name="camera_infra_1_optical_frame">
+    <inertial>
+      <origin xyz="1.52683853338331E-08 1.48608003051636E-07 -0.00158020887627678" rpy="0 0 0" />
+      <mass value="0.000453168790516429" />
+      <inertia ixx="4.84012226840139E-09" ixy="1.92888940614797E-14"
+        ixz="3.69655517006993E-13"
+        iyy="4.84044260907388E-09" iyz="1.45486421873192E-13" izz="4.34108781911687E-09" />
+    </inertial>
+    <visual>
+      <origin xyz="0 0 0" rpy="0 0 0" />
+      <geometry>
+        <mesh filename="${camera_mesh_path}camera_infra_1_optical_frame.STL" />
+      </geometry>
+      <material name="camera_sensor_material" />
+    </visual>
+    <collision>
+      <origin xyz="0 0 0" rpy="0 0 0" />
+      <geometry>
+        <mesh filename="${camera_mesh_path}camera_infra_1_optical_frame.STL" />
+      </geometry>
+    </collision>
+  </link>
+  <joint name="camera_infra_1_optical_joint" type="fixed">
+    <origin xyz="0.01587 -0.025 0.0125" rpy="-1.5707963267949 0 -1.5707963267949" />
+    <parent link="camera_bottom_screw_frame" />
+    <child link="camera_infra_1_optical_frame" />
+  </joint>
+  <!-- Infrared camera 2 frame -->
+  <link name="camera_infra2_frame">
+    <inertial>
+      <origin xyz="-0.00158020887627678 -1.52683853303637E-08 -1.48608003050581E-07" rpy="0 0 0" />
+      <mass value="0.000453168790516429" />
+      <inertia ixx="4.34108781911687E-09" ixy="-3.69655517007898E-13"
+        ixz="-1.45486421873762E-13"
+        iyy="4.84012226840139E-09" iyz="1.92888940594506E-14" izz="4.84044260907389E-09" />
+    </inertial>
+    <visual>
+      <origin xyz="0 0 0" rpy="0 0 0" />
+      <geometry>
+        <mesh filename="${camera_mesh_path}camera_infra2_frame.STL" />
+      </geometry>
+      <material name="camera_sensor_material" />
+    </visual>
+    <collision>
+      <origin xyz="0 0 0" rpy="0 0 0" />
+      <geometry>
+        <mesh filename="${camera_mesh_path}camera_infra2_frame.STL" />
+      </geometry>
+    </collision>
+  </link>
+  <joint name="camera_infra2_joint" type="fixed">
+    <origin xyz="0.01587 0.025 0.0125" rpy="0 0 0" />
+    <parent link="camera_bottom_screw_frame" />
+    <child link="camera_infra2_frame" />
+  </joint>
+  <!-- Infrared camera 2 optical frame -->
+  <link name="camera_infra2_optical_frame">
+    <inertial>
+      <origin xyz="1.52683853268942E-08 1.4860800305058E-07 -0.00158020887627678" rpy="0 0 0" />
+      <mass value="0.000453168790516429" />
+      <inertia ixx="4.84012226840139E-09" ixy="1.92888940594538E-14"
+        ixz="3.69655517007897E-13"
+        iyy="4.84044260907389E-09" iyz="1.45486421873764E-13" izz="4.34108781911687E-09" />
+    </inertial>
+    <visual>
+      <origin xyz="0 0 0" rpy="0 0 0" />
+      <geometry>
+        <mesh filename="${camera_mesh_path}camera_infra2_optical_frame.STL" />
+      </geometry>
+      <material name="camera_sensor_material" />
+    </visual>
+    <collision>
+      <origin xyz="0 0 0" rpy="0 0 0" />
+      <geometry>
+        <mesh filename="${camera_mesh_path}camera_infra2_optical_frame.STL" />
+      </geometry>
+    </collision>
+  </link>
+  <joint name="camera_infra2_optical_joint" type="fixed">
+    <origin xyz="0.01587 0.025 0.0125" rpy="-1.5707963267949 0 -1.5707963267949" />
+    <parent link="camera_bottom_screw_frame" />
+    <child link="camera_infra2_optical_frame" />
+  </joint>
+  <!-- Color camera frame -->
+  <link name="camera_color_frame">
+    <inertial>
+      <origin xyz="-0.00177079701156752 -2.20101367029782E-07 2.09893364599916E-07" rpy="0 0 0" />
+      <mass value="0.000139779365329478" />
+      <inertia ixx="6.69130695410276E-10" ixy="-1.53742421247628E-13"
+        ixz="-2.28137695085953E-14"
+        iyy="6.11277085561398E-10" iyz="4.18921196289284E-14" izz="6.11078036871936E-10" />
+    </inertial>
+    <visual>
+      <origin xyz="0 0 0" rpy="0 0 0" />
+      <geometry>
+        <mesh filename="${camera_mesh_path}camera_color_frame.STL" />
+      </geometry>
+      <material name="camera_sensor_material" />
+    </visual>
+    <collision>
+      <origin xyz="0 0 0" rpy="0 0 0" />
+      <geometry>
+        <mesh filename="${camera_mesh_path}camera_color_frame.STL" />
+      </geometry>
+    </collision>
+  </link>
+  <joint name="camera_color_joint" type="fixed">
+    <origin xyz="0.017533 0.010995 0.012505" rpy="0 0 0" />
+    <parent link="camera_bottom_screw_frame" />
+    <child link="camera_color_frame" />
+  </joint>
+  <!-- Color camera optical frame -->
+  <link name="camera_color_optical_frame">
+    <inertial>
+      <origin xyz="2.20101367029782E-07 -2.09893364599916E-07 -0.00177079701156752" rpy="0 0 0" />
+      <mass value="0.000139779365329478" />
+      <inertia ixx="6.11277085561398E-10" ixy="4.18921196289284E-14"
+        ixz="1.53742421247628E-13"
+        iyy="6.11078036871936E-10" iyz="2.28137695085953E-14" izz="6.69130695410276E-10" />
+    </inertial>
+    <visual>
+      <origin xyz="0 0 0" rpy="0 0 0" />
+      <geometry>
+        <mesh filename="${camera_mesh_path}camera_color_optical_frame.STL" />
+      </geometry>
+      <material name="camera_sensor_material" />
+    </visual>
+    <collision>
+      <origin xyz="0 0 0" rpy="0 0 0" />
+      <geometry>
+        <mesh filename="${camera_mesh_path}camera_color_optical_frame.STL" />
+      </geometry>
+    </collision>
+  </link>
+  <joint name="camera_color_optical_joint" type="fixed">
+    <origin xyz="0.017533 0.010995 0.012505" rpy="-1.5707963267949 0 -1.5707963267949" />
+    <parent link="camera_bottom_screw_frame" />
+    <child link="camera_color_optical_frame" />
+  </joint>
+  <!-- Depth camera frame -->
+  <link name="camera_depth_frame">
+    <inertial>
+      <origin xyz="-0.00158020887627678 -1.52683853338331E-08 -1.48608003051662E-07" rpy="0 0 0" />
+      <mass value="0.000453168790516429" />
+      <inertia ixx="4.34108781911687E-09" ixy="-3.69655517006982E-13"
+        ixz="-1.45486421873185E-13"
+        iyy="4.84012226840139E-09" iyz="1.92888940614707E-14" izz="4.84044260907388E-09" />
+    </inertial>
+    <visual>
+      <origin xyz="0 0 0" rpy="0 0 0" />
+      <geometry>
+        <mesh filename="${camera_mesh_path}camera_depth_frame.STL" />
+      </geometry>
+      <material name="camera_sensor_material" />
+    </visual>
+    <collision>
+      <origin xyz="0 0 0" rpy="0 0 0" />
+      <geometry>
+        <mesh filename="${camera_mesh_path}camera_depth_frame.STL" />
+      </geometry>
+    </collision>
+  </link>
+  <joint name="camera_depth_joint" type="fixed">
+    <origin xyz="0.01587 -0.025 0.0125" rpy="0 0 0" />
+    <parent link="camera_bottom_screw_frame" />
+    <child link="camera_depth_frame" />
+  </joint>
+  <!-- Depth camera optical frame -->
+  <link name="camera_depth_optical_frame">
+    <inertial>
+      <origin xyz="1.52683853338331E-08 1.4860800305165E-07 -0.00158020887627678" rpy="0 0 0" />
+      <mass value="0.000453168790516429" />
+      <inertia ixx="4.84012226840139E-09" ixy="1.9288894061467E-14" ixz="3.69655517006976E-13"
+        iyy="4.84044260907388E-09" iyz="1.454864218732E-13" izz="4.34108781911687E-09" />
+    </inertial>
+    <visual>
+      <origin xyz="0 0 0" rpy="0 0 0" />
+      <geometry>
+        <mesh filename="${camera_mesh_path}camera_depth_optical_frame.STL" />
+      </geometry>
+      <material name="camera_sensor_material" />
+    </visual>
+    <collision>
+      <origin xyz="0 0 0" rpy="0 0 0" />
+      <geometry>
+        <mesh filename="${camera_mesh_path}camera_depth_optical_frame.STL" />
+      </geometry>
+    </collision>
+  </link>
+  <joint name="camera_depth_optical_joint" type="fixed">
+    <origin xyz="0.01587 -0.025 0.0125" rpy="-1.5707963267949 0 -1.5707963267949" />
+    <parent link="camera_bottom_screw_frame" />
+    <child link="camera_depth_optical_frame" />
+  </joint>
 </robot>
